File: pcb/3xHDMI/3xHDMI.kicad_pcb (KiCad board)
At the start: 4 copper layers, 100 x 35.5 mm, 93 parts, among them J1 HDMI0-OUT, J10 SERIAL, J2 PJ-3200, J3 HDMI1-OUT, J4 HDMI2-OUT, J5 KH-TYPE-C-16P, J6 POWER_O, J7 DATA3, J8 DATA2, J9 DATA1, P1 Header-Female-2.54_1x8, Q1 AO3400, Q2 AO3400, Q3 AO3400, Q4 AO3400, Q5 AO3400, Q6 AO3400, Q7 AO3400, Q8 AO3400, Q9 AO3400, SW1 KEY, SW2 KEY, SW3 KEY, SW4 KEY, U1 CH340G, U2 AMS1117-3.3, X1 12MHz

Commit message: prep array board
Parts:
- removed C1, C2: 104, kicad_lceda:C0603
- added H1: MountingHole, MountingHole:MountingHole_3.2mm_M3, F.Cu at (211.0, 106.0)
- added H2: MountingHole, MountingHole:MountingHole_3.2mm_M3, F.Cu at (186.0, 106.0)
- added J11: Conn_01x02, Connector_PinHeader_2.54mm:PinHeader_1x02_P2.54mm_Vertical_SMD_Pin1Left, B.Cu at (201.0, 106.0)
- added SW5: KEY, kicad_lceda:SW-SMD_L6.0-W3.3-LS8.0, B.Cu at (173.0, 108.0)
- added SW6: KEY, kicad_lceda:SW-SMD_L6.0-W3.3-LS8.0, B.Cu at (173.0, 103.0)
- C11, C12, R35, R36: moved to B.Cu
- J2: value PJ-3200 -> Conn_01x02; footprint kicad_lceda:AUDIO-TH_PJ-3200 -> Connector_PinHeader_2.54mm:PinHeader_1x02_P2.54mm_Vertical_SMD_Pin1Left
- J4: value HDMI2-OUT -> HDMI2-INOUT
- R7, R8: value 3K3 -> 10K; moved to B.Cu
- moved C11 15.8 mm to (225.6, 106.0), turned to -90 degrees
- moved R35 15.8 mm to (223.8, 106.0), turned to 90 degrees
- moved J2 9.66 mm to (195.0, 106.0), turned to 0 degrees
- moved C12 7.75 mm to (219.2, 106.0), turned to -90 degrees
- moved R36 7.75 mm to (221.0, 106.0), turned to 90 degrees
- moved R7 6.86 mm to (185.0, 101.5), turned to 0 degrees
- moved R13 5.33 mm to (236.8, 100.1)
- moved J5 5.08 mm to (240.5, 105.4), turned to 0 degrees
- moved R18 4.89 mm to (243.9, 100.1), turned to 0 degrees
- moved R8 4.50 mm to (185.0, 99.5), turned to 0 degrees
Connections:
- net /AUDIO_L renamed /PL_KEY4
- net /AUDIO_R renamed /PL_KEY5
- C10 pad 1: Net-(C10-Pad1) -> Net-(J2-Pin_2)
- J2 pad 2: Net-(C1-Pad1) -> Net-(J2-Pin_2)
- J4 pad 20: Net-(C10-Pad1) -> Net-(J2-Pin_2)
- J4 pad 21: Net-(C10-Pad1) -> Net-(J2-Pin_2)
- J4 pad 22: Net-(C10-Pad1) -> Net-(J2-Pin_2)
- J4 pad 23: Net-(C10-Pad1) -> Net-(J2-Pin_2)
- P1 pad 7: +5V -> +3V3
- R34 pad 2: Net-(C10-Pad1) -> Net-(J2-Pin_2)
- R7 pad 2: Net-(C1-Pad1) -> +3V3
- R8 pad 2: Net-(C2-Pad1) -> +3V3
Routing:
- net Net-(J11-Pin_2): track 4.28 -> 35.9 mm
- net +5V: track 156.9 -> 126.0 mm
- net Net-(J2-Pin_2): track 0.00 -> 28.6 mm, vias 0 -> 1
- net Net-(C1-Pad1): track 10.5 -> 0.00 mm
- net Net-(C10-Pad1): track 7.04 -> 0.00 mm
- net Net-(C2-Pad1): track 5.85 -> 0.00 mm
- net /PL_KEY5: track 97.5 -> 91.9 mm
- net +3V3: track 250.0 -> 254.4 mm
- net GND: track 58.8 -> 62.0 mm, vias 147 -> 64
- net /PL_KEY4: track 94.2 -> 91.1 mm
- net /D-: track 19.1 -> 16.8 mm
- net Net-(C12-Pad1): track 4.03 -> 6.07 mm
- net /D+: track 18.7 -> 17.4 mm
- net Net-(J5-CC1): track 2.82 -> 3.58 mm
Other:
- board text added: "MIX"
- board text added: "MIX IS INPUT"
- board text added: "MODULATE"
- board text added: "THRU"
- board text added: "THRU IS INPUT"

Commit message: add messy graphics
Parts:
- added G***: LOGO, LOGO, B.Cu at (234.0, 93.0)
- added G***: LOGO, LOGO, B.Cu at (168.4, 93.0)
- added G***: LOGO, LOGO, B.Cu at (202.0, 93.0)
Routing:
- net /D-: track 16.8 -> 16.1 mm
- net Net-(J11-Pin_2): track 35.9 -> 35.4 mm
