File: pcb/3xHDMI/3xHDMI.kicad_sch (KiCad schematic)
At the start: 92 parts, among them J1 HDMI0-OUT, J10 SERIAL, J2 PJ-3200, J3 HDMI1-OUT, J4 HDMI2-OUT, J5 KH-TYPE-C-16P, J6 POWER_O, J7 DATA3, J8 DATA2, J9 DATA1, P1 Header-Female-2.54_1x8, Q1 AO3400, Q2 AO3400, Q3 AO3400, Q4 AO3400, Q5 AO3400, Q6 AO3400, Q7 AO3400, Q8 AO3400, Q9 AO3400, SW1 KEY, SW2 KEY, SW3 KEY, SW4 KEY, U1 CH340G, U2 AMS1117-3.3, X1 12MHz

Commit message: GOT INPUT WORKING ALRIGHTgit statusgit status
Other:
- note added: "short shield on input"

Commit message: prep array board
Parts:
- removed C1, C2: 104, kicad_lceda:C0603, symbol Device:C
- removed J2: PJ-3200, kicad_lceda:AUDIO-TH_PJ-3200, symbol kicad_lceda:PJ-3200
- added H1, H2: MountingHole, MountingHole:MountingHole_3.2mm_M3, symbol Mechanical:MountingHole
- added J11, J2: Conn_01x02, Connector_PinHeader_2.54mm:PinHeader_1x02_P2.54mm_Vertical_SMD_Pin1Left, symbol Connector_Generic:Conn_01x02
- added SW5, SW6: KEY, kicad_lceda:SW-SMD_L6.0-W3.3-LS8.0, symbol kicad_lceda:TS-1101-C-W
- J4: value HDMI2-OUT -> HDMI2-INOUT
- R7, R8: value 3K3 -> 10K; SuppliersPartNumber C22978 -> C25804
Connections:
- net +3V3: now also P1.7, R7.2, R8.2
- net +5V: no longer P1.7
- net GND: now also J11.1 (Pin_1), J2.1 (Pin_1), SW5.1, SW6.1
- net at C10.1, J4.20 (SHD), J4.21 (SHD)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: now also J2.2 (Pin_2)
- net at C11.1, J3.20 (SHD), J3.21 (SHD)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: now also J11.2 (Pin_2)
- net AUDIO_L renamed PL_KEY4
- net PL_KEY4: now also SW6.2
- net AUDIO_R renamed PL_KEY5
- net PL_KEY5: now also SW5.2
Other:
- note added: "never an input"
- moved on the sheet: R2

Commit message: Update stack up and some other clean up
Parts:
- C10, C11, C12: value 103 -> 103n
- C3, C7, C9: value 104 -> 104n
- C4, C5: value 22P -> 22p
- C6, C8: value 106 -> 106n
- J10, J6: now not fitted
- J3: value HDMI1-OUT -> HDMI1-INOUT
Changed lines of the file:
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@@
 		(on_board yes)
 		(in_pos_files yes)
-		(dnp no)
+		(dnp yes)
 		(fields_autoplaced yes)
 		(property "Reference" "J10"
@@
 			)
 		)
-		(property "Value" "104"
+		(property "Value" "104n"
 			(at 351.556 214.484 0)
 			(show_name no)
@@
 			)
 		)
-		(property "Value" "22P"
+		(property "Value" "22p"
 			(at 238.506 130.81 0)
 			(show_name no)
@@
 			)
 		)
-		(property "Value" "103"
+		(property "Value" "103n"
 			(at 49.022 53.086 0)
 			(show_name no)
@@
 			)
 		)
-		(property "Value" "22P"
+		(property "Value" "22p"
 			(at 224.536 130.81 0)
 			(show_name no)
@@
 			)
 		)
-		(property "Value" "106"
+		(property "Value" "106n"
 			(at 278.384 215.3919 0)
 			(show_name no)
@@
 		(on_board yes)
 		(in_pos_files yes)
-		(dnp no)
+		(dnp yes)
 		(fields_autoplaced yes)
 		(property "Reference" "J6"
@@
 			)
 		)
-		(property "Value" "HDMI1-OUT"
+		(property "Value" "HDMI1-INOUT"
 			(at 73.66 105.918 0)
 			(show_name no)
@@
 			)
 		)
-		(property "Value" "103"
+		(property "Value" "103n"
 			(at 50.038 129.54 0)
 			(show_name no)
@@
 			)
 		)
-		(property "Value" "104"
+		(property "Value" "104n"
 			(at 211.582 122.936 0)
 			(show_name no)
@@
 			)
 		)
-		(property "Value" "103"
+		(property "Value" "103n"
 			(at 49.276 205.994 0)
 			(show_name no)
@@
 			)
 		)
-		(property "Value" "104"
+		(property "Value" "104n"
 			(at 291.084 214.122 0)
 			(show_name no)
@@
 			)
 		)
-		(property "Value" "106"
+		(property "Value" "106n"
 			(at 337.312 215.3919 0)
 			(show_name no)
